Commit message: second_commit

File: urdf/robot_model.xacro (robot description, xacro)
@@ -19,4 +19,7 @@
         <box size="0.5 0.3 0.07" />
       </geometry>
+      <material name="white">
+        <color rgba="1.0 1.0 1.0 1.0" />
+      </material>
     </visual>
   </link>
@@ -24,22 +27,25 @@
     <inertial>
       <mass value="0.2" />
-      <origin rpy="0 0 0" xyz="0.08 0 -0.02" />
-      <inertia ixx="0.0002" ixy="0" ixz="0" iyy="0.0002" iyz="0" izz="0.0002" />
+      <origin rpy="0 0 0" xyz="0 0 0" />
+      <inertia ixx="0.000338" ixy="0" ixz="0" iyy="0.000338" iyz="0" izz="0.000338" />
     </inertial>
     <collision name="front_balance_collision">
-      <origin rpy="0 0 0" xyz="0.08 0 -0.02" />
+      <origin rpy="0 0 0" xyz="0 0 0" />
       <geometry>
-        <sphere radius="0.05" />
+        <sphere radius="0.065" />
       </geometry>
     </collision>
     <visual name="front_balance_visual">
-      <origin rpy="0 0 0" xyz="0.08 0 -0.02" />
+      <origin rpy="0 0 0" xyz="0 0 0" />
       <geometry>
-        <sphere radius="0.05" />
+        <sphere radius="0.065" />
       </geometry>
+      <material name="black">
+        <color rgba="0.0 0.0 0.0 1.0" />
+      </material>
     </visual>
   </link>
   <joint name="joint_front_balance" type="continuous">
-    <origin rpy="0 0 0" xyz="0.08 0 -0.02" />
+    <origin rpy="0 0 0" xyz="0.08 0 -0.035" />
     <child link="link_front_balance" />
     <parent link="base_link" />
@@ -60,4 +66,7 @@
           <cylinder length="0.04" radius="0.1" />
         </geometry>
+        <material name="black">
+          <color rgba="0.0 0.0 0.0 1.0" />
+        </material>
       </collision>
       <visual name="${name}_visual">
@@ -79,13 +88,13 @@
     </joint>
   </xacro:macro>
+  <xacro:link_wheel name="link_back_left_wheel" />
   <xacro:link_wheel name="link_back_right_wheel" />
-  <xacro:link_wheel name="link_back_left_wheel" />
-  <xacro:joint_wheel name="joint_back_right_wheel" child="link_back_right_wheel" origin_xyz="-0.05 0.15 0" />
-  <xacro:joint_wheel name="joint_back_left_wheel" child="link_back_left_wheel" origin_xyz="-0.05 -0.15 0" />
+  <xacro:joint_wheel name="joint_back_left_wheel" child="link_back_left_wheel" origin_xyz="-0.05 0.15 0" />
+  <xacro:joint_wheel name="joint_back_right_wheel" child="link_back_right_wheel" origin_xyz="-0.05 -0.15 0" />
   <!-- Create camera model -->
-  <link name="camera_link">
+  <link name="camera_body">
     <inertial>
       <mass value="0.1" />
-      <origin rpy="0 0 0" xyz="0 0 0.035" />
+      <origin rpy="0 0 0" xyz="0 0 0" />
       <inertia ixx="1e-4" ixy="0" ixz="0" iyy="1e-4" iyz="0" izz="0.000015" />
     </inertial>
@@ -96,17 +105,48 @@
     </collision>
     <visual>
-      <origin rpy="0 0 0" xyz="0 0 0.035" />
+      <origin rpy="0 0 0" xyz="0 0 0.05" />
       <geometry>
         <box size="0.03 0.03 0.1" />
       </geometry>
+      <material name="blue">
+        <color rgba="0 0 1 1.0" />
+      </material>
     </visual>
   </link>
-  <joint name="camera_joint" type="continuous">
+  <joint name="camera_body_joint" type="continuous">
     <origin rpy="0 0 0" xyz="0 0 0.035" />
-    <child link="camera_link" />
+    <child link="camera_body" />
     <parent link="base_link" />
     <axis xyz="0 0 1" />
     <limit effort="10000" velocity="1000" />
     <joint_properties damping="1.0" friction="1.0" />
+  </joint>
+  <link name="camera_link">
+    <inertial>
+      <mass value="1e-5" />
+      <origin xyz="0 0 0" rpy="0 0 0"/>
+      <inertia ixx="1e-6" ixy="0" ixz="0" iyy="1e-6" iyz="0" izz="1e-6" />
+    </inertial>
+    <collision>
+      <origin xyz="0 0 0.025" rpy="0 0 0"/>
+      <geometry>
+        <box size="0.03 0.03 0.01"/>
+      </geometry>
+    </collision>
+    <visual>
+      <origin xyz="0 0 0.005" rpy="0 0 0"/>
+      <geometry>
+        <box size="0.03 0.03 0.01"/>
+      </geometry>
+      <material name="blue">
+        <color rgba="0 0 1 1.0" />
+      </material>
+    </visual>
+  </link>
+  <joint name="camera_joint" type="fixed">
+    <axis xyz="0 1 0" />
+    <origin xyz="0 0 0.1" rpy="0 0 0"/>
+    <parent link="camera_body"/>
+    <child link="camera_link"/>
   </joint>
   <!-- Create transmission model -->
@@ -131,7 +171,7 @@
     </actuator>
   </transmission>
-  <transmission name="camera_link_transmission">
+  <transmission name="camera_body_transmission">
     <type>transmission_interface/SimpleTransmission</type>
-    <joint name="camera_joint">
+    <joint name="camera_body_joint">
       <hardwareInterface>hardware_interface/EffortJointInterface</hardwareInterface>
     </joint>

Commit message: Update robot_model.xacro

File: urdf/robot_model.xacro (robot description, xacro)
@@ -5,5 +5,5 @@
   <link name="base_link">
     <inertial>
-      <mass value="10" />
+      <mass value="5" />
       <origin rpy="0 0 0" xyz="0 0 0.1" />
       <inertia ixx="0.0790833" ixy="0" ixz="0" iyy="0.2124166" iyz="0" izz="0.2833333" />
